Commit message: feat: add Nav2 + slam_toolbox navigation and Ros2RobotTool.navigate
Add a 360-degree LiDAR to the robot (ray sensor -> /scan), Nav2 + slam_toolbox online-async configs and a navigation.launch.py, and route Ros2RobotTool.navigate through Nav2's NavigateToPose action. Verified end-to-end: robot navigated 0.556m toward a (0.8,0) goal. 73 tests pass.

File: ros2/src/robot_description/urdf/simple_diffbot.urdf.xacro (robot description, xacro)
@@ -101,5 +101,14 @@
     <origin xyz="0.13 0 0.02"/>
   </joint>
-  <link name="lidar_link"/>
+  <link name="lidar_link">
+    <visual>
+      <geometry><cylinder radius="0.04" length="0.03"/></geometry>
+      <material name="dark"><color rgba="0.15 0.15 0.15 1.0"/></material>
+    </visual>
+    <collision>
+      <geometry><cylinder radius="0.04" length="0.03"/></geometry>
+    </collision>
+    <xacro:cylinder_inertia m="0.05" r="0.04" l="0.03"/>
+  </link>
   <joint name="lidar_joint" type="fixed">
     <parent link="base_link"/>
@@ -142,4 +151,35 @@
     </sensor>
   </gazebo>
+  <gazebo reference="lidar_link">
+    <sensor type="ray" name="lidar">
+      <pose>0 0 0 0 0 0</pose>
+      <visualize>false</visualize>
+      <update_rate>10</update_rate>
+      <ray>
+        <scan>
+          <horizontal>
+            <samples>360</samples>
+            <resolution>1</resolution>
+            <min_angle>-3.141592653589793</min_angle>
+            <max_angle>3.141592653589793</max_angle>
+          </horizontal>
+        </scan>
+        <range>
+          <min>0.12</min>
+          <max>12.0</max>
+          <resolution>0.02</resolution>
+        </range>
+      </ray>
+      <plugin name="lidar_controller" filename="libgazebo_ros_ray_sensor.so">
+        <always_on>true</always_on>
+        <ros>
+          <namespace>/</namespace>
+          <remapping>~/out:=scan</remapping>
+        </ros>
+        <output_type>sensor_msgs/LaserScan</output_type>
+        <frame_name>lidar_link</frame_name>
+      </plugin>
+    </sensor>
+  </gazebo>
   <gazebo>
     <plugin name="diff_drive" filename="libgazebo_ros_diff_drive.so">

Commit message: fix: stabilize visual approach and add scenario regressions

File: ros2/src/robot_description/urdf/simple_diffbot.urdf.xacro (robot description, xacro)
@@ -85,4 +85,24 @@
     <origin xyz="-0.11 0 -0.04"/>
   </joint>
+  <!-- Front support prevents the camera mass from tipping the body forward. -->
+  <link name="front_caster_wheel">
+    <visual>
+      <geometry><sphere radius="0.02"/></geometry>
+      <material name="dark"/>
+    </visual>
+    <collision>
+      <geometry><sphere radius="0.02"/></geometry>
+    </collision>
+    <xacro:sphere_inertia m="0.05" r="0.02"/>
+  </link>
+  <joint name="front_caster_joint" type="fixed">
+    <parent link="base_link"/>
+    <child link="front_caster_wheel"/>
+    <origin xyz="0.11 0 -0.04"/>
+  </joint>
+  <gazebo reference="front_caster_wheel">
+    <mu1>0.01</mu1>
+    <mu2>0.01</mu2>
+  </gazebo>
   <!-- front-facing camera -->
   <link name="camera_link">
